File: output/pcbs/travipad2026.kicad_pcb (KiCad board)
At the start: 2 copper layers, 183 x 66 mm, 28 parts

Commit message: no jlc text
Other:
- board text removed: "JLCJLCJLCJLC"
Changed lines of the file:
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@@
   (title_block
     (title "travipad2026")
-    (date "2026-07-27")
+    (date "2026-07-28")
     (rev "2026.07.09")
     (company "Travis Hardiman")
@@
         (size 1 1)
         (thickness 0.15)
-      )
-    )
-  )
-  (gr_text "JLCJLCJLCJLC"
-    (at 109.97278220000001 102.1592522 -45)
-    (layer "F.SilkS" )
-    (effects
-      (font
-        (size 1 1)
-        (thickness 0.15)

Commit message: holes
Parts:
- added HOLE1: , travis:MountingHole_2.2mm_M2_Pad_Via, F.Cu at (121.0, 106.1)
- added HOLE2: , travis:MountingHole_2.2mm_M2_Pad_Via, F.Cu at (240.0, 106.1)
Other:
- board text added: "2026.08.02"
- board text removed: "2026.07.09"
Changed lines of the file:
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@@
   (title_block
     (title "travipad2026")
-    (date "2026-07-28")
-    (rev "2026.07.09")
+    (date "2026-08-02")
+    (rev "2026.08.02")
     (company "Travis Hardiman")
   )
@@
     )
   )
-  (gr_text "2026.07.09"
+  (gr_text "2026.08.02"
     (at 150.71981045 126.6074692 0)
     (layer "F.SilkS" )
@@
     )
   )
+    (module "travis:MountingHole_2.2mm_M2_Pad_Via" (layer "F.Cu")
+      (at 120.95061495 106.0660172 -45)
+      (fp_text reference "HOLE1" (at 0 -3.2) (layer "F.SilkS") hide
+        (effects (font (size 1 1) (thickness 0.15)))
+      )
+      (fp_circle (center 0 0) (end 2.45 0) (layer "F.CrtYd") (width 0.05) (fill none))
+      (pad "1" thru_hole circle locked (at 1.166726 1.166726) (size 0.7 0.7) (drill 0.4) (layers *.Cu *.Mask))
+      (pad "1" thru_hole circle locked (at 0 0) (size 4.4 4.4) (drill 2.2) (layers *.Cu *.Mask))
+      (pad "1" thru_hole circle locked (at 0 1.65) (size 0.7 0.7) (drill 0.4) (layers *.Cu *.Mask))
+      (pad "1" thru_hole circle locked (at 1.166726 -1.166726) (size 0.7 0.7) (drill 0.4) (layers *.Cu *.Mask))
+      (pad "1" thru_hole circle locked (at -1.65 0) (size 0.7 0.7) (drill 0.4) (layers *.Cu *.Mask))
+      (pad "1" thru_hole circle locked (at -1.166726 -1.166726) (size 0.7 0.7) (drill 0.4) (layers *.Cu *.Mask))
+      (pad "1" thru_hole circle locked (at -1.166726 1.166726) (size 0.7 0.7) (drill 0.4) (layers *.Cu *.Mask))
+      (pad "1" thru_hole circle locked (at 1.65 0) (size 0.7 0.7) (drill 0.4) (layers *.Cu *.Mask))
+      (pad "1" thru_hole circle locked (at 0 -1.65) (size 0.7 0.7) (drill 0.4) (layers *.Cu *.Mask))
+    )
+    (module "travis:MountingHole_2.2mm_M2_Pad_Via" (layer "F.Cu")
+      (at 240.02739685 106.0660172 -45)
+      (fp_text reference "HOLE2" (at 0 -3.2) (layer "F.SilkS") hide
+        (effects (font (size 1 1) (thickness 0.15)))
+      )
+      (fp_circle (center 0 0) (end 2.45 0) (layer "F.CrtYd") (width 0.05) (fill none))
+      (pad "2" thru_hole circle locked (at 1.166726 1.166726) (size 0.7 0.7) (drill 0.4) (layers *.Cu *.Mask))
+      (pad "2" thru_hole circle locked (at 0 0) (size 4.4 4.4) (drill 2.2) (layers *.Cu *.Mask))
+      (pad "2" thru_hole circle locked (at 0 1.65) (size 0.7 0.7) (drill 0.4) (layers *.Cu *.Mask))
+      (pad "2" thru_hole circle locked (at 1.166726 -1.166726) (size 0.7 0.7) (drill 0.4) (layers *.Cu *.Mask))
+      (pad "2" thru_hole circle locked (at -1.65 0) (size 0.7 0.7) (drill 0.4) (layers *.Cu *.Mask))
+      (pad "2" thru_hole circle locked (at -1.166726 -1.166726) (size 0.7 0.7) (drill 0.4) (layers *.Cu *.Mask))
+      (pad "2" thru_hole circle locked (at -1.166726 1.166726) (size 0.7 0.7) (drill 0.4) (layers *.Cu *.Mask))
+      (pad "2" thru_hole circle locked (at 1.65 0) (size 0.7 0.7) (drill 0.4) (layers *.Cu *.Mask))
+      (pad "2" thru_hole circle locked (at 0 -1.65) (size 0.7 0.7) (drill 0.4) (layers *.Cu *.Mask))
+    )
   (gr_line (start 119.48614879999997 138.61338719999998) (end 90.47431269480249 109.60155109480249) (layer Edge.Cuts) (stroke (width 0.15) (type default)))
 (gr_line (start 90.4743126948025 102.5304832948025) (end 117.41508100519752 75.5897149051975) (layer Edge.Cuts) (stroke (width 0.15) (type default)))

Commit message: v2 routing
Connections:
- D1 pad 1: row0 -> row1
- D10 pad 1: row1 -> row3
- D11 pad 1: row2 -> row0
- D12 pad 1: row3 -> row2
- D2 pad 1: row1 -> row3
- D3 pad 1: row2 -> row0
- D4 pad 1: row3 -> row2
- D5 pad 1: row0 -> row1
- D6 pad 1: row1 -> row3
- D7 pad 1: row2 -> row0
- D8 pad 1: row3 -> row2
- D9 pad 1: row0 -> row1
Other:
- outline, holes or cut-outs redrawn
Changed lines of the file:
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@@
       )
       (pad "1" smd roundrect (at -1.4 0 45) (size 1.25 1.75) (layers "B.Cu" "B.Paste" "B.Mask") (roundrect_rratio 0.2)
- (net 1 "row0")
+ (net 2 "row1")
       )
       (pad "2" smd roundrect (at 1.4 0 45) (size 1.25 1.75) (layers "B.Cu" "B.Paste" "B.Mask") (roundrect_rratio 0.2)
@@
       )
       (pad "1" smd roundrect (at -1.4 0 45) (size 1.25 1.75) (layers "B.Cu" "B.Paste" "B.Mask") (roundrect_rratio 0.2)
- (net 2 "row1")
+ (net 4 "row3")
       )
       (pad "2" smd roundrect (at 1.4 0 45) (size 1.25 1.75) (layers "B.Cu" "B.Paste" "B.Mask") (roundrect_rratio 0.2)
@@
       )
       (pad "1" smd roundrect (at -1.4 0 45) (size 1.25 1.75) (layers "B.Cu" "B.Paste" "B.Mask") (roundrect_rratio 0.2)
- (net 3 "row2")
+ (net 1 "row0")
       )
       (pad "2" smd roundrect (at 1.4 0 45) (size 1.25 1.75) (layers "B.Cu" "B.Paste" "B.Mask") (roundrect_rratio 0.2)
@@
       )
       (pad "1" smd roundrect (at -1.4 0 45) (size 1.25 1.75) (layers "B.Cu" "B.Paste" "B.Mask") (roundrect_rratio 0.2)
- (net 4 "row3")
+ (net 3 "row2")
       )
       (pad "2" smd roundrect (at 1.4 0 45) (size 1.25 1.75) (layers "B.Cu" "B.Paste" "B.Mask") (roundrect_rratio 0.2)
@@
       )
       (pad "1" smd roundrect (at -1.4 0 45) (size 1.25 1.75) (layers "B.Cu" "B.Paste" "B.Mask") (roundrect_rratio 0.2)
- (net 1 "row0")
+ (net 2 "row1")
       )
       (pad "2" smd roundrect (at 1.4 0 45) (size 1.25 1.75) (layers "B.Cu" "B.Paste" "B.Mask") (roundrect_rratio 0.2)
@@
       )
       (pad "1" smd roundrect (at -1.4 0 45) (size 1.25 1.75) (layers "B.Cu" "B.Paste" "B.Mask") (roundrect_rratio 0.2)
- (net 2 "row1")
+ (net 4 "row3")
       )
       (pad "2" smd roundrect (at 1.4 0 45) (size 1.25 1.75) (layers "B.Cu" "B.Paste" "B.Mask") (roundrect_rratio 0.2)
@@
       )
       (pad "1" smd roundrect (at -1.4 0 45) (size 1.25 1.75) (layers "B.Cu" "B.Paste" "B.Mask") (roundrect_rratio 0.2)
- (net 3 "row2")
+ (net 1 "row0")
       )
       (pad "2" smd roundrect (at 1.4 0 45) (size 1.25 1.75) (layers "B.Cu" "B.Paste" "B.Mask") (roundrect_rratio 0.2)
@@
       )
       (pad "1" smd roundrect (at -1.4 0 45) (size 1.25 1.75) (layers "B.Cu" "B.Paste" "B.Mask") (roundrect_rratio 0.2)
- (net 4 "row3")
+ (net 3 "row2")
       )
       (pad "2" smd roundrect (at 1.4 0 45) (size 1.25 1.75) (layers "B.Cu" "B.Paste" "B.Mask") (roundrect_rratio 0.2)
@@
       )
       (pad "1" smd roundrect (at -1.4 0 45) (size 1.25 1.75) (layers "B.Cu" "B.Paste" "B.Mask") (roundrect_rratio 0.2)
- (net 1 "row0")
+ (net 2 "row1")
       )
       (pad "2" smd roundrect (at 1.4 0 45) (size 1.25 1.75) (layers "B.Cu" "B.Paste" "B.Mask") (roundrect_rratio 0.2)
@@
       )
       (pad "1" smd roundrect (at -1.4 0 45) (size 1.25 1.75) (layers "B.Cu" "B.Paste" "B.Mask") (roundrect_rratio 0.2)
- (net 2 "row1")
+ (net 4 "row3")
       )
       (pad "2" smd roundrect (at 1.4 0 45) (size 1.25 1.75) (layers "B.Cu" "B.Paste" "B.Mask") (roundrect_rratio 0.2)
@@
       )
       (pad "1" smd roundrect (at -1.4 0 45) (size 1.25 1.75) (layers "B.Cu" "B.Paste" "B.Mask") (roundrect_rratio 0.2)
- (net 3 "row2")
+ (net 1 "row0")
       )
       (pad "2" smd roundrect (at 1.4 0 45) (size 1.25 1.75) (layers "B.Cu" "B.Paste" "B.Mask") (roundrect_rratio 0.2)
@@
       )
       (pad "1" smd roundrect (at -1.4 0 45) (size 1.25 1.75) (layers "B.Cu" "B.Paste" "B.Mask") (roundrect_rratio 0.2)
- (net 4 "row3")
+ (net 3 "row2")
       )
       (pad "2" smd roundrect (at 1.4 0 45) (size 1.25 1.75) (layers "B.Cu" "B.Paste" "B.Mask") (roundrect_rratio 0.2)
@@
     (locked no)
     (layer B.Cu)
-    (net 1)
+    (net 2)
   )
   (segment
@@
     (locked no)
     (layer B.Cu)
-    (net 2)
+    (net 4)
   )
   (segment
@@
     (locked no)
     (layer B.Cu)
-    (net 3)
+    (net 1)
   )
   (segment
@@
     (locked no)
     (layer B.Cu)
-    (net 4)
+    (net 3)
   )
   (segment
@@
     (locked no)
     (layer B.Cu)
-    (net 1)
+    (net 2)
   )
   (segment
@@
     (locked no)
     (layer B.Cu)
-    (net 2)
+    (net 4)
   )
   (segment
@@
     (locked no)
     (layer B.Cu)
-    (net 3)
+    (net 1)
   )
   (segment
@@
     (locked no)
     (layer B.Cu)
-    (net 4)
+    (net 3)
   )
   (segment
@@
     (locked no)
     (layer B.Cu)
-    (net 1)
+    (net 2)
   )
   (segment
@@
     (locked no)
     (layer B.Cu)
-    (net 2)
+    (net 4)
   )
   (segment
@@
     (locked no)
     (layer B.Cu)
-    (net 3)
+    (net 1)
   )
   (segment
@@
     (locked no)
     (layer B.Cu)
-    (net 4)
+    (net 3)
   )
   (footprint "ceoloide:utility_ergogen_logo"
@@
 (gr_line (start 228.39270990000003 130.5142341) (end 192.12369289999998 130.5142341) (layer Edge.Cuts) (stroke (width 0.15) (type default)))
 (gr_line (start 188.588159 131.97870020000002) (end 181.953472 138.6133872) (layer Edge.Cuts) (stroke (width 0.15) (type default)))
-(gr_line (start 155.7049132 140.07785330000002) (end 178.41793810000001 140.07785330000002) (layer Edge.Cuts) (stroke (width 0.15) (type default)))
-(gr_line (start 155.7049132 140.07785330000002) (end 155.7049132 130.1783584) (layer Edge.Cuts) (stroke (width 0.15) (type default)))
-(gr_line (start 155.7049132 130.1783584) (end 145.7347076 130.1783584) (layer Edge.Cuts) (stroke (width 0.15) (type default)))
-(gr_line (start 145.7347076 140.07785330000002) (end 145.7347076 130.1783584) (layer Edge.Cuts) (stroke (width 0.15) (type default)))
-(gr_line (start 123.0216827 140.07785330000002) (end 145.7347076 140.07785330000002) (layer Edge.Cuts) (stroke (width 0.15) (type default)))
+(gr_line (start 178.41793810000001 140.07785330000002) (end 123.0216827 140.07785330000002) (layer Edge.Cuts) (stroke (width 0.15) (type default)))
 (gr_arc (start 90.47431269480248 102.53048329480248) (mid 89.00984659480248 106.06601719480248) (end 90.47431269480248 109.60155109480249) (layer Edge.Cuts) (stroke (width 0.15) (type default)))
 (gr_arc (start 124.48614880519752 75.58971490519751) (mid 120.95061490519751 74.12524880519751) (end 117.41508100519751 75.58971490519751) (layer Edge.Cuts) (stroke (width 0.15) (type default)))

Commit message: logo & ground
Parts:
- turned ROC1 to 0 degrees
Routing:
- added copper zone on B.Cu, net GND
- added copper zone on F.Cu, net GND
Changed lines of the file:
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@@
       (effects (font (size 1 1) (thickness 0.1)))
+    )
+    (zone
+      (layer "F.Cu")
+      (name "eyes")
+      (hatch edge 0.5)
+      (connect_pads
+        (clearance 0)
+      )
+      (min_thickness 0.25)
+      (keepout
+        (tracks allowed)
+        (vias allowed)
+        (pads allowed)
+        (copperpour not_allowed)
+        (footprints allowed)
+      )
+      (placement
+        (enabled no)
+        (sheetname "")
+      )
+      (fill
+        (thermal_gap 0.5)
+        (thermal_bridge_width 0.5)
+        (island_removal_mode 0)
+      )
+      (polygon
+        (pts
+          (xy 209.357760 85.778761) (xy 209.357760 87.129424) (xy 211.608867 87.129424) (xy 211.608867 85.778761)
+        )
+      )
     )
     (fp_poly
@@
    )
 (module "travis:travis" (layer "B.Cu")
-    (at 210.25820134999998 91.1814195 -45)
+    (at 210.25820134999998 91.1814195 0)
     (attr virtual)
     (fp_text reference "ROC1" (at 0 -0.5 0)(layer "B.Fab") hide
@@
       (pad "2" thru_hole circle locked (at 0 -1.65) (size 0.7 0.7) (drill 0.4) (layers *.Cu *.Mask))
     )
+  (zone
+    (net 13)
+    (net_name "GND")
+    (locked no)
+    (layers "B.Cu")
+    (name "back ground")
+    (hatch edge 0.5)
+    (connect_pads yes
+      (clearance 0.508)
+    )
+    (min_thickness 0.25)
+    (filled_areas_thickness no)
+    (fill
+      yes
+      (thermal_gap 0.5)
+      (thermal_bridge_width 0.5)
+      (smoothing chamfer)
+      (radius 0.5)
+      (island_removal_mode 1)
+      (island_area_min 5)
+    )
+    (polygon
+      (pts
+        (xy 15 45) (xy 305 45) (xy 305 230) (xy 15 230)
+      )
+    )
+  )
+  (zone
+    (net 13)
+    (net_name "GND")
+    (locked no)
+    (layers "F.Cu")
+    (name "fore ground")
+    (hatch edge 0.5)
+    (connect_pads yes
+      (clearance 0.508)
+    )
+    (min_thickness 0.25)
+    (filled_areas_thickness no)
+    (fill
+      (mode hatch)
+      (thermal_gap 0.5)
+      (thermal_bridge_width 0.5)
+      (smoothing chamfer)
+      (radius 0.5)
+      (island_removal_mode 1)
+      (island_area_min 5)
+      (hatch_thickness 1)
+      (hatch_gap 1.5)
+      (hatch_orientation 45)
+      (hatch_border_algorithm hatch_thickness)
+      (hatch_min_hole_area 0.3)
+    )
+    (polygon
+      (pts
+        (xy 20 50) (xy 310 50) (xy 310 235) (xy 20 235)
+      )
+    )
+  )
   (gr_line (start 119.48614879999997 138.61338719999998) (end 90.47431269480249 109.60155109480249) (layer Edge.Cuts) (stroke (width 0.15) (type default)))
 (gr_line (start 90.4743126948025 102.5304832948025) (end 117.41508100519752 75.5897149051975) (layer Edge.Cuts) (stroke (width 0.15) (type default)))
